Commit message: Add goal manifold

File: data/r3_robot.urdf (robot description, URDF)
Before this commit: robot flexible, 5 links, 4 joints
Links:
- link link1: geometry visual cylinder length=1. radius=0.12
- link link2: geometry visual cylinder length=1. radius=0.12
- link link3: geometry visual cylinder length=1. radius=0.12
